File: m5stack_board_unitree_brushless_digital_servo.kicad_pcb (KiCad board)
At the start: 2 copper layers, 50 x 35 mm, 28 parts, among them J1 XT30UPB-M, J2 ZX-HY2.0-4PZZ, J3 B3B-PH-K-S(LF)(SN), J4 B3B-PH-K-S(LF)(SN), J5 B3B-PH-K-S(LF)(SN), J6 B3B-PH-K-S(LF)(SN), J7 B3B-PH-K-S(LF)(SN), U1 74LVC1G14, U2 XC6206P332MR, U3 74LVC1G126, U4 74LVC1G125

Commit message: Add a MINI blade fuse F1 between J1 and BAT
BAT had no protection: a short on the board or in the servo wiring would let
the battery drive a large current with nothing to break it. F1 takes a MINI
blade fuse (ISO 8820-3, 32 V, 1000 A breaking capacity), which car parts shops
in Japan sell; the fuse itself is user supplied. 15 A covers five J288 servos
(9.6 A worst case) and stays within the XT30 rating.

- Footprint: two Keystone 3557 universal clips (LCSC C2680614, wave soldered
  in Economic PCBA) 9.73 mm apart, per the Keystone layout for MINI fuses,
  bodies facing each other; pads fully connected to the pours.
- Schematic: J1 + -> BAT_IN -> F1 -> BAT -> C7 and the ports.
- Board: F1 stands just left of J1 where C7 was. BAT_IN is an F.Cu pour from
  J1 + to the top clip; the bottom clip goes straight into the B.Cu BAT band
  under the ports. C7 moves to the top strip (body 2.57 mm from the edge) and
  reaches BAT through a via into the B.Cu BAT pour, which now also runs up the
  left of F1. The board name moves to the back silkscreen.
- JLCPCB: the export lists F1 as two clips, F1A and F1B, each at the middle
  of its tails, rotated to match the EasyEDA land pattern.
- pincheck: J1 pin 2 is BAT_IN; F1 is BAT_IN / BAT.

DRC (with schematic parity), ERC and the board checks are clean.

Co-Authored-By: Claude Opus 5.5 <noreply@anthropic.com>
Claude-Session: https://claude.ai/code/session_01WJ1YBGdXpG8xhBv94Snq4Y
Parts:
- added F1: MINI 15A, Library:Fuseholder_Blade_Mini_Keystone_3557x2, F.Cu at (166.5, 125.6)
- moved C7 11.3 mm to (158.7, 115.9)
Connections:
- J1 pad 2: /BAT -> /BAT_IN
Routing:
- net /BAT: track 33.7 -> 27.8 mm, vias 0 -> 1
- net GND: track 40.6 -> 41.0 mm, vias 19 -> 18
- added copper zone on F.Cu, net /BAT_IN
