File: m5stack_board_unitree_brushless_digital_servo.kicad_pcb (KiCad board)
At the start: 2 copper layers, 50 x 35 mm, 29 parts, among them J1 XT30UPB-M, J2 ZX-HY2.0-4PZZ, J3 B3B-PH-K-S(LF)(SN), J4 B3B-PH-K-S(LF)(SN), J5 B3B-PH-K-S(LF)(SN), J6 B3B-PH-K-S(LF)(SN), J7 B3B-PH-K-S(LF)(SN), U1 74LVC1G14, U2 XC6206P332MR, U3 74LVC1G126, U4 74LVC1G125

Commit message: Use the XFCN XF-508P-B-B holder for F1
The JLCPCB order page showed no stock for the Keystone 3557 clips (C2680614),
although the parts API still listed them. F1 now uses the XFCN XF-508P-B-B
MINI blade fuse holder (C19727305, about 46k in stock): one insulated block
with both clips, 15-30 A, 500 V, wave soldered in Economic PCBA.

- Footprint from the XFCN drawing (16.0 x 6.7 x 7.35 mm body, holes
  9.80 x 3.40 mm) and the JLCPCB land pattern (2.5 mm pads, 1.8 mm holes);
  the EasyEDA STEP needs no offset.
- F1 moves 1.4 mm up and 0.6 mm right to fit between C7 and J1; the B.Cu BAT
  pour edge over F1 rises to y 116.6 and steps down clear of the top-right
  mounting hole.
- One part, so the export no longer splits F1 into F1A / F1B; its BOM
  comment says "XF-508P-B-B fuse holder (fuse not included)".
- README, AGENTS.md and the design document: the new holder, and use only
  tools/jlcpcb_export.py for the JLCPCB files (plugins and a direct board
  upload miss the per-part corrections).

DRC, ERC and the board checks are clean; the CPL check puts F1 on its pads.

Co-Authored-By: Claude Opus 5.5 <noreply@anthropic.com>
Claude-Session: https://claude.ai/code/session_01WJ1YBGdXpG8xhBv94Snq4Y
Parts:
- F1: footprint Library:Fuseholder_Blade_Mini_Keystone_3557x2 -> Library:Fuseholder_Blade_Mini_XFCN_XF-508P-B-B
- moved F1 1.54 mm to (167.1, 124.2)

Commit message: Use 470 ohm for the bleeder R4
The servo signal turned out to be 5 V logic. Its pull-up to 5 V feeds current
through R3 and, while U3 drives high, through U3 into the 3.3 V rail, which the
LDO cannot sink. The pull-up value is unknown, so R4 now drains 7 mA: enough for
pull-ups of 850 ohm or more on all five ports ((5 - 3.3) V / (Rp / 5 + 47 ohm +
about 25 ohm of U3 output)). It dissipates 23 mW of its 100 mW rating.
R4 is the Basic part C23179.

Co-Authored-By: Claude Opus 5.5 <noreply@anthropic.com>
Claude-Session: https://claude.ai/code/session_01WJ1YBGdXpG8xhBv94Snq4Y
Parts:
- R4: value 2.2k -> 470
Changed lines of the file:
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@@
 			)
 		)
-		(property "Value" "2.2k"
+		(property "Value" "470"
 			(at 0 1.43 270)
 			(layer "F.Fab")
@@
 			)
 		)
-		(property "LCSC" "C4190"
+		(property "LCSC" "C23179"
 			(at 0 0 270)
 			(layer "F.Fab")
