File: m5stack_board_unitree_brushless_digital_servo.kicad_sch (KiCad schematic)
At the start: 24 parts, among them J1 XT30UPB-M, J2 ZX-HY2.0-4PZZ, J3 B3B-PH-K-S(LF)(SN), J4 B3B-PH-K-S(LF)(SN), J5 B3B-PH-K-S(LF)(SN), J6 B3B-PH-K-S(LF)(SN), J7 B3B-PH-K-S(LF)(SN), U1 74LVC1G14, U2 XC6206P332MR, U3 74LVC1G126, U4 74LVC1G125

Commit message: Add a MINI blade fuse F1 between J1 and BAT
BAT had no protection: a short on the board or in the servo wiring would let
the battery drive a large current with nothing to break it. F1 takes a MINI
blade fuse (ISO 8820-3, 32 V, 1000 A breaking capacity), which car parts shops
in Japan sell; the fuse itself is user supplied. 15 A covers five J288 servos
(9.6 A worst case) and stays within the XT30 rating.

- Footprint: two Keystone 3557 universal clips (LCSC C2680614, wave soldered
  in Economic PCBA) 9.73 mm apart, per the Keystone layout for MINI fuses,
  bodies facing each other; pads fully connected to the pours.
- Schematic: J1 + -> BAT_IN -> F1 -> BAT -> C7 and the ports.
- Board: F1 stands just left of J1 where C7 was. BAT_IN is an F.Cu pour from
  J1 + to the top clip; the bottom clip goes straight into the B.Cu BAT band
  under the ports. C7 moves to the top strip (body 2.57 mm from the edge) and
  reaches BAT through a via into the B.Cu BAT pour, which now also runs up the
  left of F1. The board name moves to the back silkscreen.
- JLCPCB: the export lists F1 as two clips, F1A and F1B, each at the middle
  of its tails, rotated to match the EasyEDA land pattern.
- pincheck: J1 pin 2 is BAT_IN; F1 is BAT_IN / BAT.

DRC (with schematic parity), ERC and the board checks are clean.

Co-Authored-By: Claude Opus 5.5 <noreply@anthropic.com>
Claude-Session: https://claude.ai/code/session_01WJ1YBGdXpG8xhBv94Snq4Y
Parts:
- added F1: MINI 15A, Library:Fuseholder_Blade_Mini_Keystone_3557x2, symbol Device:Fuse
Connections:
- net BAT: now also F1.2; no longer J1.2 (Pin_2)
- new net BAT_IN: F1.1, J1.2 (Pin_2)
Other:
- note added: "Servo power J1: XT30 (2 = +) F1: MINI blade fuse, 15 A"
- note removed: "Servo power J1: XT30 (2 = +)"
- moved on the sheet: C7, J1
Changed lines of the file:
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@@
 	(symbol
 		(lib_id "Connector_Generic:Conn_01x02")
-		(at 30.48 142.24 180)
+		(at 25.4 142.24 180)
 		(unit 1)
 		(exclude_from_sim no)
@@
 		(dnp no)
 		(property "Reference" "J1"
-			(at 28.575 135.89 0)
+			(at 23.495 135.89 0)
 			(effects
 				(font
@@
 		)
 		(property "Value" "XT30UPB-M"
-			(at 28.575 147.32 0)
+			(at 23.495 147.32 0)
 			(effects
 				(font
@@
 		)
 		(property "Footprint" "Library:AMASS_XT30UPB-M_1x02_P5.0mm_Vertical"
-			(at 30.48 142.24 0)
+			(at 25.4 142.24 0)
 			(effects
 				(font
@@
 		)
 		(property "Datasheet" "~"
-			(at 30.48 142.24 0)
+			(at 25.4 142.24 0)
 			(effects
 				(font
@@
 		)
 		(property "LCSC" "C428721"
-			(at 30.48 142.24 0)
+			(at 25.4 142.24 0)
 			(effects
 				(font
@@
 	)
 	(symbol
+		(lib_id "Device:Fuse")
+		(at 44.45 139.7 90)
+		(unit 1)
+		(exclude_from_sim no)
+		(in_bom yes)
+		(on_board yes)
+		(dnp no)
+		(property "Reference" "F1"
+			(at 44.45 136.525 90)
+			(effects
+				(font
+					(size 1.27 1.27)
+				)
+			)
+		)
+		(property "Value" "MINI 15A"
+			(at 44.45 142.875 90)
+			(effects
+				(font
+					(size 1.27 1.27)
+				)
+			)
+		)
+		(property "Footprint" "Library:Fuseholder_Blade_Mini_Keystone_3557x2"
+			(at 44.45 139.7 0)
+			(effects
+				(font
+					(size 1.27 1.27)
+				)
+				(hide yes)
+			)
+		)
+		(property "Datasheet" "https://www.littelfuse.com/assetdocs/littelfuse_datasheet_297_mini32v.pdf"
+			(at 44.45 139.7 0)
+			(effects
+				(font
+					(size 1.27 1.27)
+				)
+				(hide yes)
+			)
+		)
+		(property "Description" "MINI blade fuse (Littelfuse 297 / Bussmann ATM, user supplied) in two Keystone 3557 clips"
+			(at 44.45 139.7 0)
+			(effects
+				(font
+					(size 1.27 1.27)
+				)
+				(hide yes)
+			)
+		)
+		(property "LCSC" "C2680614"
+			(at 44.45 139.7 0)
+			(effects
+				(font
+					(size 1.27 1.27)
+				)
+				(hide yes)
+			)
+		)
+		(pin "1"
+		)
+		(pin "2"
+		)
+		(instances
+			(project "m5stack_board_unitree_brushless_digital_servo"
+				(path "/29a88121-680b-4e5a-b555-96da8c0e0c77"
+					(reference "F1")
+					(unit 1)
+				)
+			)
+		)
+	)
+	(symbol
 		(lib_id "Device:C_Polarized")
-		(at 50.8 143.51 0)
+		(at 53.34 143.51 0)
 		(unit 1)
 		(exclude_from_sim no)
@@
 		(dnp no)
 		(property "Reference" "C7"
-			(at 52.705 142.875 0)
+			(at 55.245 142.875 0)
 			(effects
 				(font
@@
 		)
 		(property "Value" "100u 50V"
-			(at 52.705 144.78 0)
+			(at 55.245 144.78 0)
 			(effects
 				(font
@@
 		)
 		(property "Footprint" "Library:CP_Elec_6.3x7.7"
-			(at 50.8 143.51 0)
+			(at 53.34 143.51 0)
 			(effects
 				(font
@@
 		)
 		(property "Datasheet" "~"
-			(at 50.8 143.51 0)
+			(at 53.34 143.51 0)
 			(effects
 				(font
@@
 		)
 		(property "Description" "Polarized capacitor"
-			(at 50.8 143.51 0)
+			(at 53.34 143.51 0)
 			(effects
 				(font
@@
 		)
 		(property "LCSC" "C3445238"
-			(at 50.8 143.51 0)
+			(at 53.34 143.51 0)
 			(effects
 				(font
@@
 	(wire
 		(pts
-			(xy 35.56 139.7)
-			(xy 50.8 139.7)
-		)
-		(stroke
-			(width 0)
-			(type default)
-		)
-	)
-	(wire
-		(pts
-			(xy 50.8 139.7)
+			(xy 30.48 139.7)
+			(xy 40.64 139.7)
+		)
+		(stroke
+			(width 0)
+			(type default)
+		)
+	)
+	(wire
+		(pts
+			(xy 53.34 139.7)
 			(xy 243.84 139.7)
 		)
@@
 	)
 	(junction
-		(at 50.8 139.7)
+		(at 53.34 139.7)
 		(diameter 0)
 		(color 0 0 0 0)
 	)
-	(label "BAT"
-		(at 58.42 139.7 0)
+	(wire
+		(pts
+			(xy 48.26 139.7)
+			(xy 53.34 139.7)
+		)
+		(stroke
+			(width 0)
+			(type default)
+		)
+	)
+	(label "BAT_IN"
+		(at 31.75 139.7 0)
 		(fields_autoplaced yes)
 		(effects
@@
 		)
 	)
-	(wire
-		(pts
-			(xy 35.56 142.24)
-			(xy 38.1 142.24)
+	(label "BAT"
+		(at 49.53 139.7 0)
+		(fields_autoplaced yes)
+		(effects
+			(font
+				(size 1.27 1.27)
+			)
+			(justify left bottom)
+		)
+	)
+	(wire
+		(pts
+			(xy 30.48 142.24)
+			(xy 33.02 142.24)
 		)
 		(stroke
@@
 	(symbol
 		(lib_id "power:GND")
-		(at 38.1 142.24 0)
+		(at 33.02 142.24 0)
 		(unit 1)
 		(exclude_from_sim no)
@@
 		(dnp no)
 		(property "Reference" "#PWR119"
-			(at 38.1 148.59 0)
+			(at 33.02 148.59 0)
 			(effects
 				(font
@@
 		)
 		(property "Value" "GND"
-			(at 38.1 146.05 0)
+			(at 33.02 146.05 0)
 			(effects
 				(font
@@
 		)
 		(property "Footprint" ""
-			(at 38.1 142.24 0)
+			(at 33.02 142.24 0)
 			(effects
 				(font
@@
 		)
 		(property "Datasheet" ""
-			(at 38.1 142.24 0)
+			(at 33.02 142.24 0)
 			(effects
 				(font
@@
 		)
 		(property "Description" "Power symbol creates a global label with name \"GND\" , ground"
-			(at 38.1 142.24 0)
+			(at 33.02 142.24 0)
 			(effects
 				(font
@@
 	(symbol
 		(lib_id "power:GND")
-		(at 50.8 147.32 0)
+		(at 53.34 147.32 0)
 		(unit 1)
 		(exclude_from_sim no)
@@
 		(dnp no)
 		(property "Reference" "#PWR120"
-			(at 50.8 153.67 0)
+			(at 53.34 153.67 0)
 			(effects
 				(font
@@
 		)
 		(property "Value" "GND"
-			(at 50.8 151.13 0)
+			(at 53.34 151.13 0)
 			(effects
 				(font
@@
 		)
 		(property "Footprint" ""
-			(at 50.8 147.32 0)
+			(at 53.34 147.32 0)
 			(effects
 				(font
@@
 		)
 		(property "Datasheet" ""
-			(at 50.8 147.32 0)
+			(at 53.34 147.32 0)
 			(effects
 				(font
@@
 		)
 		(property "Description" "Power symbol creates a global label with name \"GND\" , ground"
-			(at 50.8 147.32 0)
+			(at 53.34 147.32 0)
 			(effects
 				(font
@@
 		)
 	)
-	(text "Servo power\nJ1: XT30 (2 = +)"
+	(text "Servo power\nJ1: XT30 (2 = +)\nF1: MINI blade fuse, 15 A"
 		(exclude_from_sim no)
 		(at 19.05 127 0)

Commit message: Use the XFCN XF-508P-B-B holder for F1
The JLCPCB order page showed no stock for the Keystone 3557 clips (C2680614),
although the parts API still listed them. F1 now uses the XFCN XF-508P-B-B
MINI blade fuse holder (C19727305, about 46k in stock): one insulated block
with both clips, 15-30 A, 500 V, wave soldered in Economic PCBA.

- Footprint from the XFCN drawing (16.0 x 6.7 x 7.35 mm body, holes
  9.80 x 3.40 mm) and the JLCPCB land pattern (2.5 mm pads, 1.8 mm holes);
  the EasyEDA STEP needs no offset.
- F1 moves 1.4 mm up and 0.6 mm right to fit between C7 and J1; the B.Cu BAT
  pour edge over F1 rises to y 116.6 and steps down clear of the top-right
  mounting hole.
- One part, so the export no longer splits F1 into F1A / F1B; its BOM
  comment says "XF-508P-B-B fuse holder (fuse not included)".
- README, AGENTS.md and the design document: the new holder, and use only
  tools/jlcpcb_export.py for the JLCPCB files (plugins and a direct board
  upload miss the per-part corrections).

DRC, ERC and the board checks are clean; the CPL check puts F1 on its pads.

Co-Authored-By: Claude Opus 5.5 <noreply@anthropic.com>
Claude-Session: https://claude.ai/code/session_01WJ1YBGdXpG8xhBv94Snq4Y
Parts:
- F1: footprint Library:Fuseholder_Blade_Mini_Keystone_3557x2 -> Library:Fuseholder_Blade_Mini_XFCN_XF-508P-B-B; LCSC C2680614 -> C19727305
Changed lines of the file:
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@@
 			)
 		)
-		(property "Footprint" "Library:Fuseholder_Blade_Mini_Keystone_3557x2"
+		(property "Footprint" "Library:Fuseholder_Blade_Mini_XFCN_XF-508P-B-B"
 			(at 44.45 139.7 0)
 			(effects
@@
 			)
 		)
-		(property "Description" "MINI blade fuse (Littelfuse 297 / Bussmann ATM, user supplied) in two Keystone 3557 clips"
+		(property "Description" "MINI blade fuse (Littelfuse 297 / Bussmann ATM, user supplied) in an XFCN XF-508P-B-B holder"
 			(at 44.45 139.7 0)
 			(effects
@@
 			)
 		)
-		(property "LCSC" "C2680614"
+		(property "LCSC" "C19727305"
 			(at 44.45 139.7 0)
 			(effects

Commit message: Use 470 ohm for the bleeder R4
The servo signal turned out to be 5 V logic. Its pull-up to 5 V feeds current
through R3 and, while U3 drives high, through U3 into the 3.3 V rail, which the
LDO cannot sink. The pull-up value is unknown, so R4 now drains 7 mA: enough for
pull-ups of 850 ohm or more on all five ports ((5 - 3.3) V / (Rp / 5 + 47 ohm +
about 25 ohm of U3 output)). It dissipates 23 mW of its 100 mW rating.
R4 is the Basic part C23179.

Co-Authored-By: Claude Opus 5.5 <noreply@anthropic.com>
Claude-Session: https://claude.ai/code/session_01WJ1YBGdXpG8xhBv94Snq4Y
Parts:
- R4: value 2.2k -> 470; LCSC C4190 -> C23179
Changed lines of the file:
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@@
 			)
 		)
-		(property "Value" "2.2k"
+		(property "Value" "470"
 			(at 133.985 160.02 0)
 			(effects
@@
 			)
 		)
-		(property "LCSC" "C4190"
+		(property "LCSC" "C23179"
 			(at 132.08 158.75 0)
 			(effects
