File: m5stack_board_unitree_brushless_digital_servo.kicad_sch (KiCad schematic)
At the start: 24 parts, among them J1 XT30UPB-M, J2 ZX-HY2.0-4PZZ, J3 B3B-PH-K-S(LF)(SN), J4 B3B-PH-K-S(LF)(SN), J5 B3B-PH-K-S(LF)(SN), J6 B3B-PH-K-S(LF)(SN), J7 B3B-PH-K-S(LF)(SN), U1 74LVC1G14, U2 AP7333-33SAG, U3 74LVC1G126, U4 74LVC1G125

Commit message: Use a Preferred Extended RB751V-40 for D1
D1 moves from the Nexperia RB751V40,115 (C553814, Extended) to the
hongjiacheng RB751V-40 (C7502691, Preferred Extended), which carries no
feeder loading fee in Economic PCBA and has more stock. The ratings match
(VF <= 0.37 V at 1 mA, IR <= 0.5 uA at 30 V, 2 pF), and the footprint is the
same.

Its JLCPCB land pattern has the cathode as pin 1 on the left, as in KiCad,
so the CPL needs no rotation (the old part had the anode as pin 1, +180).
The CPL check puts its pads within 0.11 mm of the board pads.

Co-Authored-By: Claude Opus 5.5 <noreply@anthropic.com>
Claude-Session: https://claude.ai/code/session_01WJ1YBGdXpG8xhBv94Snq4Y
Parts:
- D1: LCSC C553814 -> C7502691
Changed lines of the file:
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@@
 			)
 		)
-		(property "LCSC" "C553814"
+		(property "LCSC" "C7502691"
 			(at 54.61 66.04 0)
 			(effects

Commit message: Use the Basic part XC6206P332MR for U2
U2 was the AP7333-33SAG carried over from the DYNAMIXEL board: an Extended
part with the lowest stock in the BOM (about 16k). The Torex XC6206P332MR-G
(C5446) is a Basic part (no feeder loading fee in Economic PCBA, about 420k
in stock) and covers the few mA the logic draws (200 mA, 6 V input, stable
with the 1 uF C2 and C3).

Its pins differ (1 GND, 2 output, 3 input), so:
- the schematic uses the KiCad XC6206PxxxMR symbol (same pin positions);
- on the board, C2 + feeds pin 3, pin 1 gets a GND via above it, the +5V
  line above U2 moves up 0.45 mm to keep that via clear of its pour
  clearance, and C2 - now joins C3 -;
- the CPL keeps +180 (same land pattern orientation as before).

DRC, ERC and the board checks are clean; the README images are updated.

Co-Authored-By: Claude Opus 5.5 <noreply@anthropic.com>
Claude-Session: https://claude.ai/code/session_01WJ1YBGdXpG8xhBv94Snq4Y
Parts:
- U2: value AP7333-33SAG -> XC6206P332MR; symbol Regulator_Linear:AP7384-33SA -> Regulator_Linear:XC6206PxxxMR; LCSC C150746 -> C5446
Connections:
- net +5V: now also U2.3 (VI); no longer U2.1 (VI)
- net GND: now also U2.1 (GND); no longer U2.3 (GND)
Changed lines of the file:
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@@
 	)
 	(symbol
-		(lib_id "Regulator_Linear:AP7384-33SA")
+		(lib_id "Regulator_Linear:XC6206PxxxMR")
 		(at 101.6 154.94 0)
 		(unit 1)
@@
 			)
 		)
-		(property "Value" "AP7333-33SAG"
+		(property "Value" "XC6206P332MR"
 			(at 99.695 149.86 0)
 			(effects
@@
 			)
 		)
-		(property "Datasheet" "https://www.diodes.com/assets/Datasheets/AP7384.pdf"
+		(property "Datasheet" "https://www.torexsemi.com/file/xc6206/XC6206.pdf"
 			(at 101.6 154.94 0)
 			(effects
@@
 			)
 		)
-		(property "LCSC" "C150746"
+		(property "LCSC" "C5446"
 			(at 101.6 154.94 0)
 			(effects

Commit message: Add the servo power fuse and pre-order fixes (ordered as 062722a) (#1)
* Add a MINI blade fuse F1 between J1 and BAT

BAT had no protection: a short on the board or in the servo wiring would let
the battery drive a large current with nothing to break it. F1 takes a MINI
blade fuse (ISO 8820-3, 32 V, 1000 A breaking capacity), which car parts shops
in Japan sell; the fuse itself is user supplied. 15 A covers five J288 servos
(9.6 A worst case) and stays within the XT30 rating.

- Footprint: two Keystone 3557 universal clips (LCSC C2680614, wave soldered
  in Economic PCBA) 9.73 mm apart, per the Keystone layout for MINI fuses,
  bodies facing each other; pads fully connected to the pours.
- Schematic: J1 + -> BAT_IN -> F1 -> BAT -> C7 and the ports.
- Board: F1 stands just left of J1 where C7 was. BAT_IN is an F.Cu pour from
  J1 + to the top clip; the bottom clip goes straight into the B.Cu BAT band
  under the ports. C7 moves to the top strip (body 2.57 mm from the edge) and
  reaches BAT through a via into the B.Cu BAT pour, which now also runs up the
  left of F1. The board name moves to the back silkscreen.
- JLCPCB: the export lists F1 as two clips, F1A and F1B, each at the middle
  of its tails, rotated to match the EasyEDA land pattern.
- pincheck: J1 pin 2 is BAT_IN; F1 is BAT_IN / BAT.

DRC (with schematic parity), ERC and the board checks are clean.

Co-Authored-By: Claude Opus 5.5 <noreply@anthropic.com>
Claude-Session: https://claude.ai/code/session_01WJ1YBGdXpG8xhBv94Snq4Y

* Document the fuse

README: pin assignment, how to choose the fuse rating, specifications, BOM,
the F1A / F1B clips in the JLCPCB files and the 3D model command. Design
document: the decision and its reasons, the layout, the footprint and the
JLCPCB handling, and the protection still missing (reverse polarity, ESD).
The README images show the new layout.

Co-Authored-By: Claude Opus 5.5 <noreply@anthropic.com>
Claude-Session: https://claude.ai/code/session_01WJ1YBGdXpG8xhBv94Snq4Y

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
Parts:
- added F1: MINI 15A, Library:Fuseholder_Blade_Mini_XFCN_XF-508P-B-B, symbol Device:Fuse
- R4: value 2.2k -> 470; LCSC C4190 -> C23179
Connections:
- net BAT: now also F1.2; no longer J1.2 (Pin_2)
- new net BAT_IN: F1.1, J1.2 (Pin_2)
Other:
- note added: "Servo power J1: XT30 (2 = +) F1: MINI blade fuse, 15 A"
- note removed: "Servo power J1: XT30 (2 = +)"
- moved on the sheet: C7, J1
Changed lines of the file:
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@@
 	(symbol
 		(lib_id "Connector_Generic:Conn_01x02")
-		(at 30.48 142.24 180)
+		(at 25.4 142.24 180)
 		(unit 1)
 		(exclude_from_sim no)
@@
 		(dnp no)
 		(property "Reference" "J1"
-			(at 28.575 135.89 0)
+			(at 23.495 135.89 0)
 			(effects
 				(font
@@
 		)
 		(property "Value" "XT30UPB-M"
-			(at 28.575 147.32 0)
+			(at 23.495 147.32 0)
 			(effects
 				(font
@@
 		)
 		(property "Footprint" "Library:AMASS_XT30UPB-M_1x02_P5.0mm_Vertical"
-			(at 30.48 142.24 0)
+			(at 25.4 142.24 0)
 			(effects
 				(font
@@
 		)
 		(property "Datasheet" "~"
-			(at 30.48 142.24 0)
+			(at 25.4 142.24 0)
 			(effects
 				(font
@@
 		)
 		(property "LCSC" "C428721"
-			(at 30.48 142.24 0)
+			(at 25.4 142.24 0)
 			(effects
 				(font
@@
 	)
 	(symbol
-		(lib_id "Device:C_Polarized")
-		(at 50.8 143.51 0)
+		(lib_id "Device:Fuse")
+		(at 44.45 139.7 90)
 		(unit 1)
 		(exclude_from_sim no)
@@
 		(on_board yes)
 		(dnp no)
+		(property "Reference" "F1"
+			(at 44.45 136.525 90)
+			(effects
+				(font
+					(size 1.27 1.27)
+				)
+			)
+		)
+		(property "Value" "MINI 15A"
+			(at 44.45 142.875 90)
+			(effects
+				(font
+					(size 1.27 1.27)
+				)
+			)
+		)
+		(property "Footprint" "Library:Fuseholder_Blade_Mini_XFCN_XF-508P-B-B"
+			(at 44.45 139.7 0)
+			(effects
+				(font
+					(size 1.27 1.27)
+				)
+				(hide yes)
+			)
+		)
+		(property "Datasheet" "https://www.littelfuse.com/assetdocs/littelfuse_datasheet_297_mini32v.pdf"
+			(at 44.45 139.7 0)
+			(effects
+				(font
+					(size 1.27 1.27)
+				)
+				(hide yes)
+			)
+		)
+		(property "Description" "MINI blade fuse (Littelfuse 297 / Bussmann ATM, user supplied) in an XFCN XF-508P-B-B holder"
+			(at 44.45 139.7 0)
+			(effects
+				(font
+					(size 1.27 1.27)
+				)
+				(hide yes)
+			)
+		)
+		(property "LCSC" "C19727305"
+			(at 44.45 139.7 0)
+			(effects
+				(font
+					(size 1.27 1.27)
+				)
+				(hide yes)
+			)
+		)
+		(pin "1"
+		)
+		(pin "2"
+		)
+		(instances
+			(project "m5stack_board_unitree_brushless_digital_servo"
+				(path "/29a88121-680b-4e5a-b555-96da8c0e0c77"
+					(reference "F1")
+					(unit 1)
+				)
+			)
+		)
+	)
+	(symbol
+		(lib_id "Device:C_Polarized")
+		(at 53.34 143.51 0)
+		(unit 1)
+		(exclude_from_sim no)
+		(in_bom yes)
+		(on_board yes)
+		(dnp no)
 		(property "Reference" "C7"
-			(at 52.705 142.875 0)
+			(at 55.245 142.875 0)
 			(effects
 				(font
@@
 		)
 		(property "Value" "100u 50V"
-			(at 52.705 144.78 0)
+			(at 55.245 144.78 0)
 			(effects
 				(font
@@
 		)
 		(property "Footprint" "Library:CP_Elec_6.3x7.7"
-			(at 50.8 143.51 0)
+			(at 53.34 143.51 0)
 			(effects
 				(font
@@
 		)
 		(property "Datasheet" "~"
-			(at 50.8 143.51 0)
+			(at 53.34 143.51 0)
 			(effects
 				(font
@@
 		)
 		(property "Description" "Polarized capacitor"
-			(at 50.8 143.51 0)
+			(at 53.34 143.51 0)
 			(effects
 				(font
@@
 		)
 		(property "LCSC" "C3445238"
-			(at 50.8 143.51 0)
+			(at 53.34 143.51 0)
 			(effects
 				(font
@@
 	(wire
 		(pts
-			(xy 35.56 139.7)
-			(xy 50.8 139.7)
-		)
-		(stroke
-			(width 0)
-			(type default)
-		)
-	)
-	(wire
-		(pts
-			(xy 50.8 139.7)
+			(xy 30.48 139.7)
+			(xy 40.64 139.7)
+		)
+		(stroke
+			(width 0)
+			(type default)
+		)
+	)
+	(wire
+		(pts
+			(xy 53.34 139.7)
 			(xy 243.84 139.7)
 		)
@@
 	)
 	(junction
-		(at 50.8 139.7)
+		(at 53.34 139.7)
 		(diameter 0)
 		(color 0 0 0 0)
 	)
-	(label "BAT"
-		(at 58.42 139.7 0)
+	(wire
+		(pts
+			(xy 48.26 139.7)
+			(xy 53.34 139.7)
+		)
+		(stroke
+			(width 0)
+			(type default)
+		)
+	)
+	(label "BAT_IN"
+		(at 31.75 139.7 0)
 		(fields_autoplaced yes)
 		(effects
@@
 		)
 	)
-	(wire
-		(pts
-			(xy 35.56 142.24)
-			(xy 38.1 142.24)
+	(label "BAT"
+		(at 49.53 139.7 0)
+		(fields_autoplaced yes)
+		(effects
+			(font
+				(size 1.27 1.27)
+			)
+			(justify left bottom)
+		)
+	)
+	(wire
+		(pts
+			(xy 30.48 142.24)
+			(xy 33.02 142.24)
 		)
 		(stroke
@@
 	(symbol
 		(lib_id "power:GND")
-		(at 38.1 142.24 0)
+		(at 33.02 142.24 0)
 		(unit 1)
 		(exclude_from_sim no)
@@
 		(dnp no)
 		(property "Reference" "#PWR119"
-			(at 38.1 148.59 0)
+			(at 33.02 148.59 0)
 			(effects
 				(font
@@
 		)
 		(property "Value" "GND"
-			(at 38.1 146.05 0)
+			(at 33.02 146.05 0)
 			(effects
 				(font
@@
 		)
 		(property "Footprint" ""
-			(at 38.1 142.24 0)
+			(at 33.02 142.24 0)
 			(effects
 				(font
@@
 		)
 		(property "Datasheet" ""
-			(at 38.1 142.24 0)
+			(at 33.02 142.24 0)
 			(effects
 				(font
@@
 		)
 		(property "Description" "Power symbol creates a global label with name \"GND\" , ground"
-			(at 38.1 142.24 0)
+			(at 33.02 142.24 0)
 			(effects
 				(font
@@
 	(symbol
 		(lib_id "power:GND")
-		(at 50.8 147.32 0)
+		(at 53.34 147.32 0)
 		(unit 1)
 		(exclude_from_sim no)
@@
 		(dnp no)
 		(property "Reference" "#PWR120"
-			(at 50.8 153.67 0)
+			(at 53.34 153.67 0)
 			(effects
 				(font
@@
 		)
 		(property "Value" "GND"
-			(at 50.8 151.13 0)
+			(at 53.34 151.13 0)
 			(effects
 				(font
@@
 		)
 		(property "Footprint" ""
-			(at 50.8 147.32 0)
+			(at 53.34 147.32 0)
 			(effects
 				(font
@@
 		)
 		(property "Datasheet" ""
-			(at 50.8 147.32 0)
+			(at 53.34 147.32 0)
 			(effects
 				(font
@@
 		)
 		(property "Description" "Power symbol creates a global label with name \"GND\" , ground"
-			(at 50.8 147.32 0)
+			(at 53.34 147.32 0)
 			(effects
 				(font
@@
 		)
 	)
-	(text "Servo power\nJ1: XT30 (2 = +)"
+	(text "Servo power\nJ1: XT30 (2 = +)\nF1: MINI blade fuse, 15 A"
 		(exclude_from_sim no)
 		(at 19.05 127 0)
@@
 			)
 		)
-		(property "Value" "2.2k"
+		(property "Value" "470"
 			(at 133.985 160.02 0)
 			(effects
@@
 			)
 		)
-		(property "LCSC" "C4190"
+		(property "LCSC" "C23179"
 			(at 132.08 158.75 0)
 			(effects
